File: joystick.kicad_sch (KiCad schematic)
At the start: 4 parts, among them J1 ICS, J2 Joystick, U1 SeeeduinoXIAO

Commit message: 発注
Connections:
- net +3V3 is gone; now on net +3.3V: U1.12 (3V3)
Changed lines of the file:
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@@
     (pin "1")
   )
-  (symbol (lib_id "power:+3V3") (at 180.34 99.06 0) (unit 1)
+  (symbol (lib_id "power:+3.3V") (at 180.34 99.06 0) (unit 1)
     (in_bom yes) (on_board yes) (fields_autoplaced)
-    (property "Reference" "#PWR08" (id 0) (at 180.34 102.87 0)
+    (property "Reference" "#PWR?" (id 0) (at 180.34 102.87 0)
       (effects (font (size 1.27 1.27)) hide)
     )
-    (property "Value" "+3V3" (id 1) (at 180.34 93.98 0))
+    (property "Value" "+3.3V" (id 1) (at 180.34 93.98 0))
     (property "Footprint" "" (id 2) (at 180.34 99.06 0)
       (effects (font (size 1.27 1.27)) hide)
@@
       (reference "#PWR07") (unit 1) (value "+5V") (footprint "")
     )
-    (path "/44822897-4828-4d5a-897a-852f3e00549a"
-      (reference "#PWR08") (unit 1) (value "+3V3") (footprint "")
-    )
     (path "/a2e4c94e-39ae-42fd-9dab-71a3e646ad94"
       (reference "#PWR09") (unit 1) (value "GND") (footprint "")
     )
+    (path "/41b0b10b-8155-4677-83e9-482aa78cd31f"
+      (reference "#PWR?") (unit 1) (value "+3.3V") (footprint "")
+    )
     (path "/cfa46d4f-d382-48ed-a9b8-77555069a309"
